Commit message: Adding more gaits.

File: resources/robots/a1/urdf/a1_biped.urdf (robot description, URDF)
Before this commit: robot a1_description, 23 links, 22 joints
Links:
- link RL_foot: geometry collision sphere radius=0.02; visual box size=0.06 0.04 0.01
Joints:
- joint RL_foot_joint: axis (none) -> 0 1 0; limit (none) -> lower=0 upper=1.5 effort=55 velocity=28.6
- joint RR_foot_joint: axis (none) -> 0 1 0; limit (none) -> lower=0 upper=1.5 effort=55 velocity=28.6

Commit message: Blind walking on uneven terrain

File: resources/robots/a1/urdf/a1_biped.urdf (robot description, URDF)
Before this commit: robot a1_description, 23 links, 22 joints
Links:
- link RL_foot: geometry collision sphere radius=0.02; visual sphere radius=0.01
